File: $Eurorack-JP6-filter.sch (KiCad schematic (older format))
At the start: 138 parts, among them J1 JACK_MONO_SW, J2 JACK_MONO_SW, J3 JACK_MONO_SW, J4 JACK_MONO_SW, J5 JACK_MONO_SW, J6 JACK_MONO_SW, P1 CONN_02X05, Q1 BCM857BS, Q2 BCM857BS, Q3 J112, Q4 J112, Q5 J112, Q6 J112, SW1 KS-01Q, U1 TL072-, U10 CD4027, U11 CD40106, U2 TL072-, U3 TL072-, U4 TL072-, U5 LM13700, U6 LM13700, U7 LM13700, U8 DG409, U9 CD4052

Commit message: started placing components, pots, jacks, sw1 and LEDs placed
Parts:
- VR6: footprint synth:RD901F-ALPHA-POT -> synth:RV16A-41-JRL
Changed lines of the file:
@@
 F 0 "VR6" H 2350 10600 50  0000 C CNN
 F 1 "50K" H 2350 10670 50  0000 C CNN
-F 2 "synth:RD901F-ALPHA-POT" H 2350 10750 60  0001 C CNN
+F 2 "synth:RV16A-41-JRL" H 2350 10750 60  0001 C CNN
 F 3 "" H 2350 10750 60  0000 C CNN
 	1    2350 10750

Commit message: placing components, a few footprints updated
Parts:
- C18, C25, C6, C7: footprint MyModules:SM0603-C-JRL -> MyModules:CAP-BOX-PFR-5MM
- R66, R67: footprint MyModules:SM0603-R-JRL -> MyModules:SM0805-HAND
Changed lines of the file:
@@
 F 0 "C6" H 8350 11800 50  0000 L CNN
 F 1 "330pF" H 8350 11600 50  0000 L CNN
-F 2 "MyModules:SM0603-C-JRL" H 8300 11700 60  0001 C CNN
+F 2 "MyModules:CAP-BOX-PFR-5MM" H 8300 11700 60  0001 C CNN
 F 3 "" H 8300 11700 60  0000 C CNN
 	1    8300 11700
@@
 F 0 "C7" H 10950 11800 50  0000 L CNN
 F 1 "330pF" H 10950 11600 50  0000 L CNN
-F 2 "MyModules:SM0603-C-JRL" H 10900 11700 60  0001 C CNN
+F 2 "MyModules:CAP-BOX-PFR-5MM" H 10900 11700 60  0001 C CNN
 F 3 "" H 10900 11700 60  0000 C CNN
 	1    10900 11700
@@
 F 0 "C18" H 16650 11800 50  0000 L CNN
 F 1 "330pF" H 16650 11600 50  0000 L CNN
-F 2 "MyModules:SM0603-C-JRL" H 16600 11700 60  0001 C CNN
+F 2 "MyModules:CAP-BOX-PFR-5MM" H 16600 11700 60  0001 C CNN
 F 3 "" H 16600 11700 60  0000 C CNN
 	1    16600 11700
@@
 F 0 "C25" H 19250 11800 50  0000 L CNN
 F 1 "330pF" H 19250 11600 50  0000 L CNN
-F 2 "MyModules:SM0603-C-JRL" H 19200 11700 60  0001 C CNN
+F 2 "MyModules:CAP-BOX-PFR-5MM" H 19200 11700 60  0001 C CNN
 F 3 "" H 19200 11700 60  0000 C CNN
 	1    19200 11700
@@
 F 0 "R66" V 18680 1400 50  0000 C CNN
 F 1 "10" V 18520 1400 50  0000 C CNN
-F 2 "MyModules:SM0603-R-JRL" H 18600 1400 60  0001 C CNN
+F 2 "MyModules:SM0805-HAND" H 18600 1400 60  0001 C CNN
 F 3 "" H 18600 1400 60  0000 C CNN
 	1    18600 1400
@@
 F 0 "R67" V 18680 2300 50  0000 C CNN
 F 1 "10" V 18520 2300 50  0000 C CNN
-F 2 "MyModules:SM0603-R-JRL" H 18600 2300 60  0001 C CNN
+F 2 "MyModules:SM0805-HAND" H 18600 2300 60  0001 C CNN
 F 3 "" H 18600 2300 60  0000 C CNN
 	1    18600 2300
