File: Eurorack-JP6-filter.kicad_pcb (KiCad board)
At the start: 2 copper layers, 65 x 100 mm, 138 parts, among them J1 JACK_MONO_SW, J2 JACK_MONO_SW, J3 JACK_MONO_SW, J4 JACK_MONO_SW, J5 JACK_MONO_SW, J6 JACK_MONO_SW, P1 CONN_02X05, Q1 BCM857BS, Q2 BCM857BS, Q3 J112, Q4 J112, Q5 J112, Q6 J112, SW1 KS-01Q, U1 TL072-, U10 CD4027, U11 CD40106, U2 TL072-, U3 TL072-, U4 TL072-, U5 LM13700, U6 LM13700, U7 LM13700, U8 DG409, U9 CD4052

Commit message: finished routing, mostly cleaned upk, parts modelled in 5365
Parts:
- Q1, Q2: footprint synth:SOT363-JRL -> MyModules:SOT363-JRL
- U5, U6, U7, U8: footprint synth:SO16-JRL -> MyModules:SO16-JRL
- VR1, VR2, VR3, VR4, VR6: footprint synth:RV16A-41-JRL -> MyModules:RV16A-41-JRL
Routing:
- net +12V: track 522.6 -> 528.4 mm
- net Net-(C3-Pad1): track 63.7 -> 60.7 mm
- net GND: track 15.9 -> 18.7 mm, vias 10 -> 12
- net Net-(R48-Pad1): track 29.5 -> 32.2 mm
- net -12V: track 284.9 -> 286.1 mm
- net SWX1: track 19.7 -> 20.6 mm
- net Net-(R4-Pad2): track 74.3 -> 73.7 mm
- net Net-(C11-Pad1): track 32.7 -> 33.4 mm
- net Net-(J4-Pad3): track 73.3 -> 73.9 mm
