File: Eurorack-JP6-filter.sch (KiCad schematic (older format))
At the start: 152 parts, among them J1 JACK_MONO_SW, J2 JACK_MONO_SW, J3 JACK_MONO_SW, J4 JACK_MONO_SW, J5 JACK_MONO_SW, J6 JACK_MONO_SW, P1 CONN_02X05, Q1 BCM857BS, Q2 BCM857BS, Q3 J112, Q4 J112, Q5 J112, Q6 J112, SW1 KS-01Q, U1 TL072-, U10 CD4027, U11 CD40106, U12 TS321, U13 TS321, U2 TL072-, U3 TL072-, U4 TL072-, U5 LM13700, U6 LM13700, U7 LM13700, U8 DG409, U9 CD4052

Commit message: v1.3 routed
Parts:
- J1, J2, J3, J4, J5, J6: footprint MyModules:PJ-301B-JACK -> MyModules:PJ-301B-JACK-SLOTS
- Q1, Q2: footprint MyModules:SOT363-JRL -> SMD TRAN:sot323-6
Connections:
- net at VR4.2: now also R3.2; no longer U1.5 (+)
- net at J3.3, VR4.3: no longer R76.2
- net at VR3.2: now also U1.5 (+); no longer R3.2
- net at J2.3, VR3.3: now also R76.2
Other:
- moved on the sheet: J2, J3, VR3, VR4
Changed lines of the file:
@@
 F 0 "Q2" H 9725 2850 60  0000 R CNN
 F 1 "BCM857BS" H 10075 2400 60  0000 R CNN
-F 2 "MyModules:SOT363-JRL" H 9225 2600 60  0001 C CNN
+F 2 "SMD TRAN:sot323-6" H 9225 2600 60  0001 C CNN
 F 3 "" H 9225 2600 60  0000 C CNN
 	1    9425 2600
@@
 L POT_US VR4
 U 1 1 553D9840
-P 2950 1900
-F 0 "VR4" H 2950 1750 50  0000 C CNN
-F 1 "50K" H 2950 1820 50  0000 C CNN
-F 2 "MyModules:RV16A-41-JRL" H 2950 1900 60  0001 C CNN
-F 3 "" H 2950 1900 60  0000 C CNN
-	1    2950 1900
+P 5375 2750
+F 0 "VR4" H 5375 2600 50  0000 C CNN
+F 1 "50K" H 5375 2670 50  0000 C CNN
+F 2 "MyModules:RV16A-41-JRL" H 5375 2750 60  0001 C CNN
+F 3 "" H 5375 2750 60  0000 C CNN
+	1    5375 2750
 	0    1    -1   0
 $EndComp
@@
 L JACK_MONO_SW J3
 U 1 1 553D99DC
-P 2200 1275
-F 0 "J3" H 1650 1175 60  0000 C CNN
-F 1 "JACK_MONO_SW" H 1950 1475 60  0000 C CNN
-F 2 "MyModules:PJ-301B-JACK" H 2100 1275 60  0001 C CNN
-F 3 "" H 2100 1275 60  0000 C CNN
-	1    2200 1275
+P 4275 2650
+F 0 "J3" H 3725 2550 60  0000 C CNN
+F 1 "JACK_MONO_SW" H 4025 2850 60  0000 C CNN
+F 2 "MyModules:PJ-301B-JACK-SLOTS" H 4175 2650 60  0001 C CNN
+F 3 "" H 4175 2650 60  0000 C CNN
+	1    4275 2650
 	1    0    0    1
 $EndComp
@@
 L POT_US VR3
 U 1 1 553DA311
-P 5375 2750
-F 0 "VR3" H 5375 2600 50  0000 C CNN
-F 1 "50K" H 5375 2670 50  0000 C CNN
-F 2 "MyModules:RV16A-41-JRL" H 5375 2750 60  0001 C CNN
-F 3 "" H 5375 2750 60  0000 C CNN
-	1    5375 2750
+P 2950 1900
+F 0 "VR3" H 2950 1750 50  0000 C CNN
+F 1 "50K" H 2950 1820 50  0000 C CNN
+F 2 "MyModules:RV16A-41-JRL" H 2950 1900 60  0001 C CNN
+F 3 "" H 2950 1900 60  0000 C CNN
+	1    2950 1900
 	0    1    -1   0
 $EndComp
@@
 L JACK_MONO_SW J2
 U 1 1 553DA31F
-P 4275 2650
-F 0 "J2" H 3725 2550 60  0000 C CNN
-F 1 "JACK_MONO_SW" H 4025 2850 60  0000 C CNN
-F 2 "MyModules:PJ-301B-JACK" H 4175 2650 60  0001 C CNN
-F 3 "" H 4175 2650 60  0000 C CNN
-	1    4275 2650
+P 2200 1275
+F 0 "J2" H 1650 1175 60  0000 C CNN
+F 1 "JACK_MONO_SW" H 1950 1475 60  0000 C CNN
+F 2 "MyModules:PJ-301B-JACK-SLOTS" H 2100 1275 60  0001 C CNN
+F 3 "" H 2100 1275 60  0000 C CNN
+	1    2200 1275
 	1    0    0    1
 $EndComp
@@
 F 0 "Q1" H 6650 6550 60  0000 R CNN
 F 1 "BCM857BS" H 7000 6100 60  0000 R CNN
-F 2 "MyModules:SOT363-JRL" H 6150 6300 60  0001 C CNN
+F 2 "SMD TRAN:sot323-6" H 6150 6300 60  0001 C CNN
 F 3 "" H 6150 6300 60  0000 C CNN
 	1    6350 6300
@@
 F 0 "J5" H 675 11975 60  0000 C CNN
 F 1 "JACK_MONO_SW" H 975 12275 60  0000 C CNN
-F 2 "MyModules:PJ-301B-JACK" H 1125 12075 60  0001 C CNN
+F 2 "MyModules:PJ-301B-JACK-SLOTS" H 1125 12075 60  0001 C CNN
 F 3 "" H 1125 12075 60  0000 C CNN
 	1    1225 12075
@@
 F 0 "J4" H 675 11025 60  0000 C CNN
 F 1 "JACK_MONO_SW" H 975 11325 60  0000 C CNN
-F 2 "MyModules:PJ-301B-JACK" H 1125 11125 60  0001 C CNN
+F 2 "MyModules:PJ-301B-JACK-SLOTS" H 1125 11125 60  0001 C CNN
 F 3 "" H 1125 11125 60  0000 C CNN
 	1    1225 11125
@@
 F 0 "J6" H 15550 15350 60  0000 C CNN
 F 1 "JACK_MONO_SW" H 15850 15650 60  0000 C CNN
-F 2 "MyModules:PJ-301B-JACK" H 16000 15450 60  0001 C CNN
+F 2 "MyModules:PJ-301B-JACK-SLOTS" H 16000 15450 60  0001 C CNN
 F 3 "" H 16000 15450 60  0000 C CNN
 	1    16100 15450
@@
 F 0 "J1" H 2025 7350 60  0000 C CNN
 F 1 "JACK_MONO_SW" H 2325 7650 60  0000 C CNN
-F 2 "MyModules:PJ-301B-JACK" H 2475 7450 60  0001 C CNN
+F 2 "MyModules:PJ-301B-JACK-SLOTS" H 2475 7450 60  0001 C CNN
 F 3 "" H 2475 7450 60  0000 C CNN
 	1    2575 7450

Commit message: fixed cretnious things only a cretin would do
Connections:
- net +12V: no longer R1.1
- net -12V: now also R1.2
- net GND: now also VR2.1; no longer VR2.3
- new net: R1.1, VR2.3
Other:
- moved on the sheet: R1
Changed lines of the file:
@@
 $EndComp
 $Comp
-L -12V #PWR018
-U 1 1 553E08DE
-P 3625 6700
-F 0 "#PWR018" H 3625 6550 50  0001 C CNN
-F 1 "-12V" H 3625 6840 50  0000 C CNN
-F 2 "" H 3625 6700 60  0000 C CNN
-F 3 "" H 3625 6700 60  0000 C CNN
-	1    3625 6700
-	1    0    0    1
-$EndComp
-$Comp
 L R_US R21
 U 1 1 553E08E4
@@
 L GND #PWR023
 U 1 1 553E2A4E
-P 2425 6500
-F 0 "#PWR023" H 2425 6250 50  0001 C CNN
-F 1 "GND" H 2425 6400 50  0000 C CNN
-F 2 "" H 2425 6500 60  0000 C CNN
-F 3 "" H 2425 6500 60  0000 C CNN
-	1    2425 6500
+P 2025 6025
+F 0 "#PWR023" H 2025 5775 50  0001 C CNN
+F 1 "GND" H 2025 5925 50  0000 C CNN
+F 2 "" H 2025 6025 60  0000 C CNN
+F 3 "" H 2025 6025 60  0000 C CNN
+	1    2025 6025
 	1    0    0    -1
 $EndComp
@@
 L R_US R1
 U 1 1 553E2C63
-P 2425 5700
-F 0 "R1" V 2505 5700 50  0000 C CNN
-F 1 "10K" V 2345 5700 50  0000 C CNN
-F 2 "MyModules:SM0603-R-JRL" H 2425 5700 60  0001 C CNN
-F 3 "" H 2425 5700 60  0000 C CNN
-	1    2425 5700
+P 2425 6675
+F 0 "R1" V 2505 6675 50  0000 C CNN
+F 1 "10K" V 2345 6675 50  0000 C CNN
+F 2 "MyModules:SM0603-R-JRL" H 2425 6675 60  0001 C CNN
+F 3 "" H 2425 6675 60  0000 C CNN
+	1    2425 6675
 	-1   0    0    -1
 $EndComp
 $Comp
-L +12V #PWR024
-U 1 1 553E321C
-P 2425 5500
-F 0 "#PWR024" H 2425 5350 50  0001 C CNN
-F 1 "+12V" H 2425 5640 50  0000 C CNN
-F 2 "" H 2425 5500 60  0000 C CNN
-F 3 "" H 2425 5500 60  0000 C CNN
-	1    2425 5500
-	1    0    0    -1
-$EndComp
-$Comp
 L R_US R9
 U 1 1 553E34C0
@@
 	4650 5600 4700 5600
 Wire Wire Line
-	2425 6400 2425 6500
-Wire Wire Line
-	2425 5900 2425 6000
+	2425 6400 2425 6475
 Wire Wire Line
 	5100 5600 5100 6350
@@
 	9775 7800 12775 7800
 Wire Wire Line
-	12775 7800 12775 7200
+	12775 7200 12775 7800
 Wire Wire Line
 	12075 7800 12075 8000
@@
 Text Notes 3825 4125 0    60   ~ 0
 FREQUENCY
-Text Notes 2200 6750 0    60   ~ 0
+Text Notes 2150 5725 0    60   ~ 0
 RESONANCE
 Text Notes 1875 925  0    60   ~ 0
@@
 	0    1    1    0
 $EndComp
+$Comp
+L -12V #PWR018
+U 1 1 553E08DE
+P 3625 6700
+F 0 "#PWR018" H 3625 6550 50  0001 C CNN
+F 1 "-12V" H 3625 6840 50  0000 C CNN
+F 2 "" H 3625 6700 60  0000 C CNN
+F 3 "" H 3625 6700 60  0000 C CNN
+	1    3625 6700
+	1    0    0    1
+$EndComp
+$Comp
+L -12V #PWR?
+U 1 1 580DC9B5
+P 2425 6950
+F 0 "#PWR?" H 2425 6800 50  0001 C CNN
+F 1 "-12V" H 2425 7090 50  0000 C CNN
+F 2 "" H 2425 6950 60  0000 C CNN
+F 3 "" H 2425 6950 60  0000 C CNN
+	1    2425 6950
+	1    0    0    1
+$EndComp
+Wire Wire Line
+	2425 6875 2425 6950
+Wire Wire Line
+	2425 6000 2425 5800
+Wire Wire Line
+	2425 5800 2025 5800
+Wire Wire Line
+	2025 5800 2025 6025
 $EndSCHEMATC
